File: ADS131M08_Arduino.kicad_sch (KiCad schematic)
At the start: 12 parts, among them J1 Power, J2 Digital/PWM, J3 Analog, J4 Digital/PWM, J5 Conn_02x12_Odd_Even, U1 ADS131M08IPB, X1 SiT8008

Commit message: Updated to use resistor arrays
Parts:
- added C10, C11, C12, C13, C6, C7, C8, C9: 10nF, Capacitor_SMD:C_0603_1608Metric, symbol Device:C_Small
- added C14, C15, C16, C17: 1uF, symbol Device:C_Small
- added RN1, RN2, RN3, RN4: 10kR, Resistor_SMD:R_Array_Concave_4x0402, symbol Device:R_Pack04
- added U2, U3: XC6206PxxxMR, Package_TO_SOT_SMD:SOT-23-3, symbol Regulator_Linear:XC6206PxxxMR
- X1: LCSC (none) -> C802854
Connections:
- net *10: now also U1.18 (~{DRDY}); no longer U1.17 (~{CS})
- net *9: now also U1.17 (~{CS}); no longer U1.16 (~{RESET}/~{SYNC})
- net +5V: now also J5.1 (Pin_1), C14.1, C16.1, U2.3 (VI), U3.3 (VI)
- net 8: now also U1.16 (~{RESET}/~{SYNC}); no longer U1.18 (~{DRDY})
- net GND: now also J5.21 (Pin_21), J5.22 (Pin_22), J5.3 (Pin_3), J5.4 (Pin_4), C14.2, C15.2, C16.2, C17.2, U2.1 (GND), U3.1 (GND)
- net IN0+: now also RN3.4 (R4.1)
- net IN0-: now also RN3.3 (R3.1)
- net IN1+: now also RN3.2 (R2.1)
- net IN1-: now also RN3.1 (R1.1)
- net IN2+: now also RN1.4 (R4.1)
- net IN2-: now also RN1.3 (R3.1)
- net IN3+: now also RN1.2 (R2.1)
- net IN3-: now also RN1.1 (R1.1)
- net IN4+: now also RN2.4 (R4.1)
- net IN4-: now also RN2.3 (R3.1)
- net IN5+: now also RN2.2 (R2.1)
- net IN5-: now also RN2.1 (R1.1)
- net IN6+: now also RN4.4 (R4.1)
- net IN6-: now also RN4.3 (R3.1)
- net IN7+: now also RN4.2 (R2.1)
- net IN7-: now also RN4.1 (R1.1)
- net +3.3V: now reaches C1.1, U1.26 (DVDD)
- net +3.3V: now also C15.1, U2.2 (VO)
- net +3.3VADC: now reaches C2.1, U1.15 (AVDD)
- net +3.3VADC: now also C17.1, U3.2 (VO)
- net Antialiasing/ADC+ renamed AIN0P
- net AIN0P: now also C6.1, RN3.5 (R4.2)
- net Antialiasing/ADC- renamed AIN0N
- net AIN0N: now also C6.2, RN3.6 (R3.2)
- net Antialiasing1/ADC+ renamed AIN1P
- net AIN1P: now also C7.1, RN3.7 (R2.2)
- net Antialiasing1/ADC- renamed AIN1N
- net AIN1N: now also C7.2, RN3.8 (R1.2)
- net Antialiasing2/ADC+ renamed AIN2P
- net AIN2P: now also C8.1, RN1.5 (R4.2)
- net Antialiasing2/ADC- renamed AIN2N
- net AIN2N: now also C8.2, RN1.6 (R3.2)
- net Antialiasing3/ADC+ renamed AIN3P
- net AIN3P: now also C9.1, RN1.7 (R2.2)
- net Antialiasing3/ADC- renamed AIN3N
- net AIN3N: now also C9.2, RN1.8 (R1.2)
- net Antialiasing4/ADC+ renamed AIN4P
- net AIN4P: now also C10.1, RN2.5 (R4.2)
- net Antialiasing4/ADC- renamed AIN4N
- net AIN4N: now also C10.2, RN2.6 (R3.2)
- net Antialiasing5/ADC+ renamed AIN5P
- net AIN5P: now also C11.1, RN2.7 (R2.2)
- net Antialiasing5/ADC- renamed AIN5N
- net AIN5N: now also C11.2, RN2.8 (R1.2)
- net Antialiasing6/ADC+ renamed AIN6P
- net AIN6P: now also C12.1, RN4.5 (R4.2)
- net Antialiasing6/ADC- renamed AIN6N
- net AIN6N: now also C12.2, RN4.6 (R3.2)
- net Antialiasing7/ADC+ renamed AIN7P
- net AIN7P: now also C13.1, RN4.7 (R2.2)
- net Antialiasing7/ADC- renamed AIN7N
- net AIN7N: now also C13.2, RN4.8 (R1.2)
- no-connect marks 2 -> 3
Other:
- removed sheet Antialiasing
- removed sheet Antialiasing1
- removed sheet Antialiasing2
- removed sheet Antialiasing3
- removed sheet Antialiasing4
- removed sheet Antialiasing5
- removed sheet Antialiasing6
- removed sheet Antialiasing7

Commit message: Commit nov 9 2024
Parts:
- added Q1, Q2, Q3: Q_NMOS_GSD, symbol Device:Q_NMOS_GSD
- added R1: 5.1kR, symbol Device:R_Small_US
- added R2: I am slightly larger resistor, symbol Device:R_Small_US
- C1, C14, C15, C16, C17, C2: footprint (none) -> Capacitor_SMD:C_0402_1005Metric; LCSC (none) -> C528974
- C10, C11, C12, C13, C6, C7, C8, C9: footprint Capacitor_SMD:C_0603_1608Metric -> Capacitor_SMD:C_0402_1005Metric; LCSC (none) -> C3855387
- C3, C5: footprint (none) -> Capacitor_SMD:C_0402_1005Metric; LCSC (none) -> C77020
- C4: footprint (none) -> Capacitor_SMD:C_0402_1005Metric; LCSC (none) -> C126524
- J5: LCSC (none) -> C2897432
- RN1, RN2, RN4: LCSC (none) -> C136853
- U1: LCSC (none) -> C2685451
Connections:
- net *11: now also U1.19 (SCLK); no longer U1.21 (DIN)
- net +3.3V: now also C5.1, X1.4 (VDD)
- net +5V: now also J5.24 (Pin_24); no longer J5.1 (Pin_1)
- net 13: now also U1.21 (DIN); no longer U1.19 (SCLK)
- net A0: now also J5.23 (Pin_23)
- net AIN0N: now also RN3.3 (R3.1); no longer RN3.6 (R3.2)
- net AIN0P: now also RN3.4 (R4.1); no longer RN3.5 (R4.2)
- net AIN1N: now also RN3.2 (R2.1); no longer RN3.8 (R1.2)
- net AIN1P: now also RN3.1 (R1.1); no longer RN3.7 (R2.2)
- net AIN2N: now also RN1.3 (R3.1); no longer RN1.6 (R3.2)
- net AIN2P: now also RN1.4 (R4.1); no longer RN1.5 (R4.2)
- net AIN3N: now also RN1.2 (R2.1); no longer RN1.8 (R1.2)
- net AIN3P: now also RN1.1 (R1.1); no longer RN1.7 (R2.2)
- net AIN4N: now also RN2.3 (R3.1); no longer RN2.6 (R3.2)
- net AIN4P: now also RN2.4 (R4.1); no longer RN2.5 (R4.2)
- net AIN5N: now also RN2.2 (R2.1); no longer RN2.8 (R1.2)
- net AIN5P: now also RN2.1 (R1.1); no longer RN2.7 (R2.2)
- net AIN6N: now also RN4.3 (R3.1); no longer RN4.6 (R3.2)
- net AIN6P: now also RN4.4 (R4.1); no longer RN4.5 (R4.2)
- net AIN7N: now also RN4.2 (R2.1); no longer RN4.8 (R1.2)
- net AIN7P: now also RN4.1 (R1.1); no longer RN4.7 (R2.2)
- net GND: now also Q1.2 (S), Q2.2 (S), Q3.2 (S), R2.2
- net IN0+: now also RN3.5 (R4.2); no longer RN3.4 (R4.1)
- net IN0-: now also RN3.6 (R3.2); no longer RN3.3 (R3.1)
- net IN1+: now also RN3.7 (R2.2); no longer RN3.2 (R2.1)
- net IN1-: now also RN3.8 (R1.2); no longer RN3.1 (R1.1)
- net IN2+: now also RN1.5 (R4.2); no longer RN1.4 (R4.1)
- net IN2-: now also RN1.6 (R3.2); no longer RN1.3 (R3.1)
- net IN3+: now also RN1.7 (R2.2); no longer RN1.2 (R2.1)
- net IN3-: now also RN1.8 (R1.2); no longer RN1.1 (R1.1)
- net IN4+: now also RN2.5 (R4.2); no longer RN2.4 (R4.1)
- net IN4-: now also RN2.6 (R3.2); no longer RN2.3 (R3.1)
- net IN5+: now also RN2.7 (R2.2); no longer RN2.2 (R2.1)
- net IN5-: now also RN2.8 (R1.2); no longer RN2.1 (R1.1)
- net IN6+: now also RN4.5 (R4.2); no longer RN4.4 (R4.1)
- net IN6-: now also RN4.6 (R3.2); no longer RN4.3 (R3.1)
- net IN7+: now also RN4.7 (R2.2); no longer RN4.2 (R2.1)
- net IN7-: now also RN4.8 (R1.2); no longer RN4.1 (R1.1)
- net SCL/A5: now also J5.2 (Pin_2); no longer J3.6 (Pin_6)
- net SDA/A4: now also J5.1 (Pin_1); no longer J3.5 (Pin_5)
- net VCC: now also R1.1
- new net: Q1.3 (D), Q2.3 (D), Q3.3 (D)
- new net SCL: R1.2, R2.1
- no-connect marks 3 -> 5
Other:
- note added: "C5383094"
- note added: "Display"
- note added: "Master"
- note added: "Sensor"
- note added: "Treat me like a voltage divider and you will see that the voltage here is still quite quite quite close to VCC!"
- moved on the sheet: RN3
